Commit message: fix urdf

File: src/gz_main/urdf/Rover.xacro (robot description, xacro)
@@ -1,25 +1,25 @@
 <?xml version="1.0" ?>
 <robot name="Rover" xmlns:xacro="http://www.ros.org/wiki/xacro">
-<xacro:include filename="$(find Rover_description)/urdf/materials.xacro" />
-<xacro:include filename="$(find Rover_description)/urdf/Rover.trans" />
-<xacro:include filename="$(find Rover_description)/urdf/Rover.gazebo" />
+<xacro:include filename="$(find gz_main)/urdf/materials.xacro" />
+<xacro:include filename="$(find gz_main)/urdf/Rover.trans" />
+<xacro:include filename="$(find gz_main)/urdf/Rover.gazebo" />
 <link name="dummy_base_link"></link>
 <link name="base_link">
   <inertial>
-    <origin xyz="-6.106915349179497e-13 -0.02576797376370591 0.3408721287496551" rpy="0 0 0"/>
+    <origin xyz="-6.106915349179497e-13 -0.02576797376370591 0.3408721287496551" rpy="0 0 -1.57"/>
     <mass value="119.00094541166615"/>
     <inertia ixx="11.367893" iyy="2.895706" izz="13.361019" ixy="-0.0" iyz="0.11269" ixz="-0.0"/>
   </inertial>
   <visual>
-    <origin xyz="0 0 0" rpy="0 0 0"/>
-    <geometry>
-      <mesh filename="file://$(find Rover_description)/meshes/base_link.stl" scale="0.001 0.001 0.001"/>
-    </geometry>
-    <material name="silver"/>
-  </visual>
-  <collision>
-    <origin xyz="0 0 0" rpy="0 0 0"/>
-    <geometry>
-      <mesh filename="file://$(find Rover_description)/meshes/base_link.stl" scale="0.001 0.001 0.001"/>
+    <origin xyz="0 0 0" rpy="0 0 1.57"/>
+    <geometry>
+      <mesh filename="file://$(find gz_main)/meshes/base_link.stl" scale="0.001 0.001 0.001"/>
+    </geometry>
+    <material name="silver"/>
+  </visual>
+  <collision>
+    <origin xyz="0 0 0" rpy="0 0 1.57"/>
+    <geometry>
+      <mesh filename="file://$(find gz_main)/meshes/base_link.stl" scale="0.001 0.001 0.001"/>
     </geometry>
   </collision>
@@ -32,14 +32,14 @@
   </inertial>
   <visual>
-    <origin xyz="0.35 0.491042 -0.196191" rpy="0 0 0"/>
-    <geometry>
-      <mesh filename="file://$(find Rover_description)/meshes/fr_wheel_1.stl" scale="0.001 0.001 0.001"/>
-    </geometry>
-    <material name="silver"/>
-  </visual>
-  <collision>
-    <origin xyz="0.35 0.491042 -0.196191" rpy="0 0 0"/>
-    <geometry>
-      <mesh filename="file://$(find Rover_description)/meshes/fr_wheel_1.stl" scale="0.001 0.001 0.001"/>
+    <origin xyz="0.45 0.491042 -0.196191" rpy="0 0 0"/>
+    <geometry>
+      <mesh filename="file://$(find gz_main)/meshes/fr_wheel_1.stl" scale="0.001 0.001 0.001"/>
+    </geometry>
+    <material name="silver"/>
+  </visual>
+  <collision>
+    <origin xyz="0.45 0.491042 -0.196191" rpy="0 0 0"/>
+    <geometry>
+      <mesh filename="file://$(find gz_main)/meshes/fr_wheel_1.stl" scale="0.001 0.001 0.001"/>
     </geometry>
   </collision>
@@ -52,14 +52,14 @@
   </inertial>
   <visual>
-    <origin xyz="0.35 0.051042 -0.196191" rpy="0 0 0"/>
-    <geometry>
-      <mesh filename="file://$(find Rover_description)/meshes/mr_wheel_1.stl" scale="0.001 0.001 0.001"/>
-    </geometry>
-    <material name="silver"/>
-  </visual>
-  <collision>
-    <origin xyz="0.35 0.051042 -0.196191" rpy="0 0 0"/>
-    <geometry>
-      <mesh filename="file://$(find Rover_description)/meshes/mr_wheel_1.stl" scale="0.001 0.001 0.001"/>
+    <origin xyz="0.45 0.051042 -0.196191" rpy="0 0 0"/>
+    <geometry>
+      <mesh filename="file://$(find gz_main)/meshes/mr_wheel_1.stl" scale="0.001 0.001 0.001"/>
+    </geometry>
+    <material name="silver"/>
+  </visual>
+  <collision>
+    <origin xyz="0.45 0.051042 -0.196191" rpy="0 0 0"/>
+    <geometry>
+      <mesh filename="file://$(find gz_main)/meshes/mr_wheel_1.stl" scale="0.001 0.001 0.001"/>
     </geometry>
   </collision>
@@ -72,14 +72,14 @@
   </inertial>
   <visual>
-    <origin xyz="0.35 -0.388958 -0.196191" rpy="0 0 0"/>
-    <geometry>
-      <mesh filename="file://$(find Rover_description)/meshes/br_wheel_1.stl" scale="0.001 0.001 0.001"/>
-    </geometry>
-    <material name="silver"/>
-  </visual>
-  <collision>
-    <origin xyz="0.35 -0.388958 -0.196191" rpy="0 0 0"/>
-    <geometry>
-      <mesh filename="file://$(find Rover_description)/meshes/br_wheel_1.stl" scale="0.001 0.001 0.001"/>
+    <origin xyz="0.45 -0.388958 -0.196191" rpy="0 0 0"/>
+    <geometry>
+      <mesh filename="file://$(find gz_main)/meshes/br_wheel_1.stl" scale="0.001 0.001 0.001"/>
+    </geometry>
+    <material name="silver"/>
+  </visual>
+  <collision>
+    <origin xyz="0.45 -0.388958 -0.196191" rpy="0 0 0"/>
+    <geometry>
+      <mesh filename="file://$(find gz_main)/meshes/br_wheel_1.stl" scale="0.001 0.001 0.001"/>
     </geometry>
   </collision>
@@ -92,14 +92,14 @@
   </inertial>
   <visual>
-    <origin xyz="-0.35 0.491042 -0.196191" rpy="0 0 0"/>
-    <geometry>
-      <mesh filename="file://$(find Rover_description)/meshes/fl_wheel_1.stl" scale="0.001 0.001 0.001"/>
-    </geometry>
-    <material name="silver"/>
-  </visual>
-  <collision>
-    <origin xyz="-0.35 0.491042 -0.196191" rpy="0 0 0"/>
-    <geometry>
-      <mesh filename="file://$(find Rover_description)/meshes/fl_wheel_1.stl" scale="0.001 0.001 0.001"/>
+    <origin xyz="-0.45 0.491042 -0.196191" rpy="0 0 0"/>
+    <geometry>
+      <mesh filename="file://$(find gz_main)/meshes/fl_wheel_1.stl" scale="0.001 0.001 0.001"/>
+    </geometry>
+    <material name="silver"/>
+  </visual>
+  <collision>
+    <origin xyz="-0.45 0.491042 -0.196191" rpy="0 0 0"/>
+    <geometry>
+      <mesh filename="file://$(find gz_main)/meshes/fl_wheel_1.stl" scale="0.001 0.001 0.001"/>
     </geometry>
   </collision>
@@ -112,14 +112,14 @@
   </inertial>
   <visual>
-    <origin xyz="-0.35 0.051042 -0.196191" rpy="0 0 0"/>
-    <geometry>
-      <mesh filename="file://$(find Rover_description)/meshes/ml_wheel_1.stl" scale="0.001 0.001 0.001"/>
-    </geometry>
-    <material name="silver"/>
-  </visual>
-  <collision>
-    <origin xyz="-0.35 0.051042 -0.196191" rpy="0 0 0"/>
-    <geometry>
-      <mesh filename="file://$(find Rover_description)/meshes/ml_wheel_1.stl" scale="0.001 0.001 0.001"/>
+    <origin xyz="-0.45 0.051042 -0.196191" rpy="0 0 0"/>
+    <geometry>
+      <mesh filename="file://$(find gz_main)/meshes/ml_wheel_1.stl" scale="0.001 0.001 0.001"/>
+    </geometry>
+    <material name="silver"/>
+  </visual>
+  <collision>
+    <origin xyz="-0.45 0.051042 -0.196191" rpy="0 0 0"/>
+    <geometry>
+      <mesh filename="file://$(find gz_main)/meshes/ml_wheel_1.stl" scale="0.001 0.001 0.001"/>
     </geometry>
   </collision>
@@ -132,18 +132,18 @@
   </inertial>
   <visual>
-    <origin xyz="-0.35 -0.388958 -0.196191" rpy="0 0 0"/>
-    <geometry>
-      <mesh filename="file://$(find Rover_description)/meshes/bl_wheel_1.stl" scale="0.001 0.001 0.001"/>
-    </geometry>
-    <material name="silver"/>
-  </visual>
-  <collision>
-    <origin xyz="-0.35 -0.388958 -0.196191" rpy="0 0 0"/>
-    <geometry>
-      <mesh filename="file://$(find Rover_description)/meshes/bl_wheel_1.stl" scale="0.001 0.001 0.001"/>
-    </geometry>
-  </collision>
-</link>
-<link name="cam_link_1">
+    <origin xyz="-0.45 -0.388958 -0.196191" rpy="0 0 0"/>
+    <geometry>
+      <mesh filename="file://$(find gz_main)/meshes/bl_wheel_1.stl" scale="0.001 0.001 0.001"/>
+    </geometry>
+    <material name="silver"/>
+  </visual>
+  <collision>
+    <origin xyz="-0.45 -0.388958 -0.196191" rpy="0 0 0"/>
+    <geometry>
+      <mesh filename="file://$(find gz_main)/meshes/bl_wheel_1.stl" scale="0.001 0.001 0.001"/>
+    </geometry>
+  </collision>
+</link>
+<!-- <link name="cam_link_1">
   <inertial>
     <origin xyz="0.0023214284363409377 6.917077683965545e-07 0.03267816705539389" rpy="0 0 0"/>
@@ -154,5 +154,5 @@
     <origin xyz="-0.0 0.562258 -0.451191" rpy="0 0 0"/>
     <geometry>
-      <mesh filename="file://$(find Rover_description)/meshes/cam_link_1.stl" scale="0.001 0.001 0.001"/>
+      <mesh filename="file://$(find gz_main)/meshes/cam_link_1.stl" scale="0.001 0.001 0.001"/>
     </geometry>
     <material name="silver"/>
@@ -161,5 +161,5 @@
     <origin xyz="-0.0 0.562258 -0.451191" rpy="0 0 0"/>
     <geometry>
-      <mesh filename="file://$(find Rover_description)/meshes/cam_link_1.stl" scale="0.001 0.001 0.001"/>
+      <mesh filename="file://$(find gz_main)/meshes/cam_link_1.stl" scale="0.001 0.001 0.001"/>
     </geometry>
   </collision>
@@ -174,5 +174,5 @@
     <origin xyz="-0.02 0.562251 -0.501191" rpy="0 0 0"/>
     <geometry>
-      <mesh filename="file://$(find Rover_description)/meshes/cam_1.stl" scale="0.001 0.001 0.001"/>
+      <mesh filename="file://$(find gz_main)/meshes/cam_1.stl" scale="0.001 0.001 0.001"/>
     </geometry>
     <material name="silver"/>
@@ -181,8 +181,8 @@
     <origin xyz="-0.02 0.562251 -0.501191" rpy="0 0 0"/>
     <geometry>
-      <mesh filename="file://$(find Rover_description)/meshes/cam_1.stl" scale="0.001 0.001 0.001"/>
-    </geometry>
-  </collision>
-</link>
+      <mesh filename="file://$(find gz_main)/meshes/cam_1.stl" scale="0.001 0.001 0.001"/>
+    </geometry>
+  </collision>
+</link> -->
 <joint name="dummy" type="fixed">
   <origin xyz="0.0 0.0 0.0" rpy="0 0 0"/>
@@ -191,5 +191,5 @@
 </joint>
 <joint name="frw_to_body" type="continuous">
-  <origin xyz="-0.35 -0.491042 0.196191" rpy="0 0 0"/>
+  <origin xyz="0.491042 -0.35  0.196191" rpy="0 0 -1.57"/>
   <parent link="base_link"/>
   <child link="fr_wheel_1"/>
@@ -197,5 +197,5 @@
 </joint>
 <joint name="mrw_to_body" type="continuous">
-  <origin xyz="-0.35 -0.051042 0.196191" rpy="0 0 0"/>
+  <origin xyz="0.051042 -0.35  0.196191" rpy="0 0 -1.57"/>
   <parent link="base_link"/>
   <child link="mr_wheel_1"/>
@@ -203,5 +203,5 @@
 </joint>
 <joint name="brw_to_body" type="continuous">
-  <origin xyz="-0.35 0.388958 0.196191" rpy="0 0 0"/>
+  <origin xyz="-0.388958 -0.35  0.196191" rpy="0 0 -1.57"/>
   <parent link="base_link"/>
   <child link="br_wheel_1"/>
@@ -209,22 +209,22 @@
 </joint>
 <joint name="flw_to_body" type="continuous">
-  <origin xyz="0.35 -0.491042 0.196191" rpy="0 0 0"/>
+  <origin xyz="0.491042 0.35  0.196191" rpy="0 0 -1.57"/>
   <parent link="base_link"/>
   <child link="fl_wheel_1"/>
-  <axis xyz="1.0 0.0 0.0"/>
+  <axis xyz="-1.0 0.0 0.0"/>
 </joint>
 <joint name="mlw_to_body" type="continuous">
-  <origin xyz="0.35 -0.051042 0.196191" rpy="0 0 0"/>
+  <origin xyz="0.051042 0.35  0.196191" rpy="0 0 -1.57"/>
   <parent link="base_link"/>
   <child link="ml_wheel_1"/>
-  <axis xyz="1.0 0.0 0.0"/>
+  <axis xyz="-1.0 0.0 0.0"/>
 </joint>
 <joint name="blw_to_body" type="continuous">
-  <origin xyz="0.35 0.388958 0.196191" rpy="0 0 0"/>
+  <origin xyz="-0.388958 0.35  0.196191" rpy="0 0 -1.57"/>
   <parent link="base_link"/>
   <child link="bl_wheel_1"/>
-  <axis xyz="1.0 0.0 0.0"/>
-</joint>
-<joint name="camlink_to_body" type="continuous">
+  <axis xyz="-1.0 0.0 0.0"/>
+</joint>
+<!-- <joint name="camlink_to_body" type="continuous">
   <origin xyz="0.0 -0.562258 0.451191" rpy="0 0 0"/>
   <parent link="base_link"/>
@@ -237,4 +237,4 @@
   <child link="cam_1"/>
   <axis xyz="1.0 0.000341 0.0"/>
-</joint>
+</joint> -->
 </robot>

Commit message: camera add

File: src/gz_main/urdf/Rover.xacro (robot description, xacro)
@@ -145,10 +145,5 @@
   </collision>
 </link>
-<!-- <link name="cam_link_1">
-  <inertial>
-    <origin xyz="0.0023214284363409377 6.917077683965545e-07 0.03267816705539389" rpy="0 0 0"/>
-    <mass value="0.023310617489636382"/>
-    <inertia ixx="8e-06" iyy="8e-06" izz="2e-06" ixy="-0.0" iyz="-0.0" ixz="-1e-06"/>
-  </inertial>
+<link name="cam_link_1">
   <visual>
     <origin xyz="-0.0 0.562258 -0.451191" rpy="0 0 0"/>
@@ -158,19 +153,8 @@
     <material name="silver"/>
   </visual>
-  <collision>
-    <origin xyz="-0.0 0.562258 -0.451191" rpy="0 0 0"/>
-    <geometry>
-      <mesh filename="file://$(find gz_main)/meshes/cam_link_1.stl" scale="0.001 0.001 0.001"/>
-    </geometry>
-  </collision>
 </link>
 <link name="cam_1">
-  <inertial>
-    <origin xyz="-0.016571501440010395 -0.026721074701518743 1.695522619860057e-05" rpy="0 0 0"/>
-    <mass value="0.04317333055495183"/>
-    <inertia ixx="6e-06" iyy="2.9e-05" izz="3.2e-05" ixy="-3e-06" iyz="0.0" ixz="0.0"/>
-  </inertial>
-  <visual>
-    <origin xyz="-0.02 0.562251 -0.501191" rpy="0 0 0"/>
+  <visual>
+    <origin xyz="-0.02 0.562251 -0.501191" rpy="0.785 0 0"/>
     <geometry>
       <mesh filename="file://$(find gz_main)/meshes/cam_1.stl" scale="0.001 0.001 0.001"/>
@@ -178,11 +162,27 @@
     <material name="silver"/>
   </visual>
-  <collision>
-    <origin xyz="-0.02 0.562251 -0.501191" rpy="0 0 0"/>
-    <geometry>
-      <mesh filename="file://$(find gz_main)/meshes/cam_1.stl" scale="0.001 0.001 0.001"/>
-    </geometry>
-  </collision>
-</link> -->
+</link>
+<gazebo reference="cam_1">
+  <sensor name="camera" type="camera">
+    <always_on>true</always_on>
+    <visualize>true</visualize>
+    <update_rate>30</update_rate>
+    <topic>camera/image</topic>
+    <!-- <gz_frame_id>cam_link_1</gz_frame_id> -->
+    <camera name="camera">
+      <camera_info_topic>camera/camera_info</camera_info_topic>
+      <horizontal_fov>1.8</horizontal_fov>
+      <image>
+        <format>R8G8B8</format>
+        <width>1920</width>
+        <height>1080</height>
+      </image>
+      <clip>
+        <near>0.1</near>
+        <far>5</far>
+      </clip>
+    </camera>
+  </sensor>
+</gazebo>
 <joint name="dummy" type="fixed">
   <origin xyz="0.0 0.0 0.0" rpy="0 0 0"/>
@@ -226,5 +226,5 @@
   <axis xyz="-1.0 0.0 0.0"/>
 </joint>
-<!-- <joint name="camlink_to_body" type="continuous">
+<joint name="camlink_to_body" type="fixed">
   <origin xyz="0.0 -0.562258 0.451191" rpy="0 0 0"/>
   <parent link="base_link"/>
@@ -232,9 +232,9 @@
   <axis xyz="0.0 -0.0 1.0"/>
 </joint>
-<joint name="cam_to_camlink" type="continuous">
+<joint name="cam_to_camlink" type="fixed">
   <origin xyz="0.02 7e-06 0.05" rpy="0 0 0"/>
   <parent link="cam_link_1"/>
   <child link="cam_1"/>
   <axis xyz="1.0 0.000341 0.0"/>
-</joint> -->
+</joint>
 </robot>

Commit message: camera pos fix

File: src/gz_main/urdf/Rover.xacro (robot description, xacro)
@@ -147,7 +147,8 @@
 <link name="cam_link_1">
   <visual>
-    <origin xyz="-0.0 0.562258 -0.451191" rpy="0 0 0"/>
-    <geometry>
-      <mesh filename="file://$(find gz_main)/meshes/cam_link_1.stl" scale="0.001 0.001 0.001"/>
+    <origin xyz="0 0 0" rpy="0 0 0"/>
+    <geometry>
+      <cylinder radius="0.01" length="0.2"/>
+      <!-- <mesh filename="file://$(find gz_main)/meshes/cam_link_1.stl" scale="0.001 0.001 0.001"/> -->
     </geometry>
     <material name="silver"/>
@@ -156,9 +157,10 @@
 <link name="cam_1">
   <visual>
-    <origin xyz="-0.02 0.562251 -0.501191" rpy="0.785 0 0"/>
-    <geometry>
-      <mesh filename="file://$(find gz_main)/meshes/cam_1.stl" scale="0.001 0.001 0.001"/>
-    </geometry>
-    <material name="silver"/>
+    <origin xyz="0 0 0" rpy="0 0 0"/>
+    <geometry>
+      <box size="0.03 0.1 0.03"/>
+    </geometry>
+    <material name="silver">
+    </material>
   </visual>
 </link>
@@ -227,14 +229,12 @@
 </joint>
 <joint name="camlink_to_body" type="fixed">
-  <origin xyz="0.0 -0.562258 0.451191" rpy="0 0 0"/>
+  <origin xyz="0.6 0 0.5" rpy="0 0 0"/>
   <parent link="base_link"/>
   <child link="cam_link_1"/>
-  <axis xyz="0.0 -0.0 1.0"/>
 </joint>
 <joint name="cam_to_camlink" type="fixed">
-  <origin xyz="0.02 7e-06 0.05" rpy="0 0 0"/>
+  <origin xyz="0 0 0.1" rpy="0 0 0"/>
   <parent link="cam_link_1"/>
   <child link="cam_1"/>
-  <axis xyz="1.0 0.000341 0.0"/>
 </joint>
 </robot>

Commit message: add planners

File: src/gz_main/urdf/Rover.xacro (robot description, xacro)
@@ -16,5 +16,7 @@
       <mesh filename="file://$(find gz_main)/meshes/base_link.stl" scale="0.001 0.001 0.001"/>
     </geometry>
-    <material name="silver"/>
+    <material name="ok">
+      <color rgba="0.4 0.4 0.4 1.0"/>
+    </material>
   </visual>
   <collision>
@@ -36,5 +38,7 @@
       <mesh filename="file://$(find gz_main)/meshes/fr_wheel_1.stl" scale="0.001 0.001 0.001"/>
     </geometry>
-    <material name="silver"/>
+    <material name="blue">
+      <color rgba="0.1 0.1 0.1 1.0"/>
+    </material>
   </visual>
   <collision>
@@ -56,5 +60,7 @@
       <mesh filename="file://$(find gz_main)/meshes/mr_wheel_1.stl" scale="0.001 0.001 0.001"/>
     </geometry>
-    <material name="silver"/>
+    <material name="blue">
+      <color rgba="0.1 0.1 0.1 1.0"/>
+    </material>
   </visual>
   <collision>
@@ -76,5 +82,5 @@
       <mesh filename="file://$(find gz_main)/meshes/br_wheel_1.stl" scale="0.001 0.001 0.001"/>
     </geometry>
-    <material name="silver"/>
+    <material name="blue"/>
   </visual>
   <collision>
@@ -96,5 +102,5 @@
       <mesh filename="file://$(find gz_main)/meshes/fl_wheel_1.stl" scale="0.001 0.001 0.001"/>
     </geometry>
-    <material name="silver"/>
+    <material name="blue"/>
   </visual>
   <collision>
@@ -116,5 +122,5 @@
       <mesh filename="file://$(find gz_main)/meshes/ml_wheel_1.stl" scale="0.001 0.001 0.001"/>
     </geometry>
-    <material name="silver"/>
+    <material name="blue"/>
   </visual>
   <collision>
@@ -136,5 +142,5 @@
       <mesh filename="file://$(find gz_main)/meshes/bl_wheel_1.stl" scale="0.001 0.001 0.001"/>
     </geometry>
-    <material name="silver"/>
+    <material name="blue"/>
   </visual>
   <collision>
